Commit message: Improve quadruped gait and controls

File: projects/07_quadruped_wheel_leg_robot/src/quadruped_wheel_leg/urdf/wheel_leg_quadruped.urdf (robot description, URDF)
Before this commit: robot wheel_leg_quadruped, 16 links, 15 joints
Links:
- added link front_left_hip_abduction_link, mass 0.28; visual sphere radius=0.060
- added link front_right_hip_abduction_link, mass 0.28; visual sphere radius=0.060
- added link rear_left_hip_abduction_link, mass 0.28; visual sphere radius=0.060
- added link rear_right_hip_abduction_link, mass 0.28; visual sphere radius=0.060
- link base_link: mass None -> 8.50
- link front_left_lower_leg_link: mass None -> 0.32
- link front_left_upper_leg_link: mass None -> 0.42
- link front_left_wheel_link: mass None -> 0.26
- link front_right_lower_leg_link: mass None -> 0.32
- link front_right_upper_leg_link: mass None -> 0.42
- link front_right_wheel_link: mass None -> 0.26
- link head_link: mass None -> 0.80
- link rear_left_lower_leg_link: mass None -> 0.32
- link rear_left_upper_leg_link: mass None -> 0.42
- link rear_left_wheel_link: mass None -> 0.26
- link rear_right_lower_leg_link: mass None -> 0.32
- link rear_right_upper_leg_link: mass None -> 0.42
- link rear_right_wheel_link: mass None -> 0.26
- link sensor_mast_link: mass None -> 0.45
Joints:
- added joint front_left_hip_abduction_joint: type revolute, parent base_link, child front_left_hip_abduction_link, origin xyz=0.28 0.22 -0.06 rpy=0 0 0, axis 1 0 0, limit lower=-0.55 upper=0.55 effort=24.0 velocity=4.5
- added joint front_right_hip_abduction_joint: type revolute, parent base_link, child front_right_hip_abduction_link, origin xyz=0.28 -0.22 -0.06 rpy=0 0 0, axis 1 0 0, limit lower=-0.55 upper=0.55 effort=24.0 velocity=4.5
- added joint rear_left_hip_abduction_joint: type revolute, parent base_link, child rear_left_hip_abduction_link, origin xyz=-0.28 0.22 -0.06 rpy=0 0 0, axis 1 0 0, limit lower=-0.55 upper=0.55 effort=24.0 velocity=4.5
- added joint rear_right_hip_abduction_joint: type revolute, parent base_link, child rear_right_hip_abduction_link, origin xyz=-0.28 -0.22 -0.06 rpy=0 0 0, axis 1 0 0, limit lower=-0.55 upper=0.55 effort=24.0 velocity=4.5
- joint front_left_hip_joint: origin xyz=0.28 0.22 -0.06 rpy=0 0 0 -> xyz=0 0 0 rpy=0 0 0; parent base_link -> front_left_hip_abduction_link
- joint front_right_hip_joint: origin xyz=0.28 -0.22 -0.06 rpy=0 0 0 -> xyz=0 0 0 rpy=0 0 0; parent base_link -> front_right_hip_abduction_link
- joint rear_left_hip_joint: origin xyz=-0.28 0.22 -0.06 rpy=0 0 0 -> xyz=0 0 0 rpy=0 0 0; parent base_link -> rear_left_hip_abduction_link
- joint rear_right_hip_joint: origin xyz=-0.28 -0.22 -0.06 rpy=0 0 0 -> xyz=0 0 0 rpy=0 0 0; parent base_link -> rear_right_hip_abduction_link

Commit message: Add quadruped drive modes and treaded wheels

File: projects/07_quadruped_wheel_leg_robot/src/quadruped_wheel_leg/urdf/wheel_leg_quadruped.urdf (robot description, URDF)
Before this commit: robot wheel_leg_quadruped, 20 links, 19 joints
Links:
- link front_left_wheel_link: geometry visual box size=0.018 0.070 0.060; visual box size=0.018 0.070 0.060
- link front_right_wheel_link: geometry visual box size=0.018 0.070 0.060; visual box size=0.018 0.070 0.060
- link rear_left_wheel_link: geometry visual box size=0.018 0.070 0.060; visual box size=0.018 0.070 0.060
- link rear_right_wheel_link: geometry visual box size=0.018 0.070 0.060; visual box size=0.018 0.070 0.060
